Commit message: Added Softhand gripper bigger reformate of code to allow for no gripper, RG6 or Softhand softhand is controlled with direct joints movement as gears were failing for so many joints added new URDFs ans SRDFs for all three versions of the robot

File: src/ur10e_simulator/UR10e_meshes/ur10e_rg6.urdf (robot description, URDF)
Before this commit: robot ur10e_robot, 25 links, 24 joints
Links:
- added link airskin_10, mass 0; collision mesh filename=package://UR10e_meshes/meshes/airskin/collision/airskin_10.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; visual mesh filename=package://UR10e_meshes/meshes/airskin/visual/airskin_10.obj
- added link gripper_link, mass 0
- added link jaws_link, mass 0
- added link left_inner_finger, mass 0.05; collision mesh filename=package://UR10e_meshes/meshes/rg6/collision/left_inner_fing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; visual mesh filename=package://UR10e_meshes/meshes/rg6/visual/left_inner_finger.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
- added link left_inner_knuckle, mass 0.05; collision mesh filename=package://UR10e_meshes/meshes/rg6/collision/left_inner_knuc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; visual mesh filename=package://UR10e_meshes/meshes/rg6/visual/left_inner_knuckle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
- added link left_outer_knuckle, mass 0.05; collision mesh filename=package://UR10e_meshes/meshes/rg6/collision/left_outer_knuc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; visual mesh filename=package://UR10e_meshes/meshes/rg6/visual/left_outer_knuckle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
- added link onrobot_rg6_base_link, mass 0.7; collision mesh filename=package://UR10e_meshes/meshes/rg6/collision/onrobot_rg6_bas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; visual mesh filename=package://UR10e_meshes/meshes/rg6/visual/onrobot_rg6_base_l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
- added link right_inner_finger, mass 0.05; collision mesh filename=package://UR10e_meshes/meshes/rg6/collision/inner_finger.obj; visual mesh filename=package://UR10e_meshes/meshes/rg6/visual/inner_finger.obj
- added link right_inner_knuckle, mass 0.05; collision mesh filename=package://UR10e_meshes/meshes/rg6/collision/inner_knuckle.o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; visual mesh filename=package://UR10e_meshes/meshes/rg6/visual/inner_knuckle.obj
- added link right_outer_knuckle, mass 0.05; collision mesh filename=package://UR10e_meshes/meshes/rg6/collision/outer_knuckle.o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; visual mesh filename=package://UR10e_meshes/meshes/rg6/visual/outer_knuckle.obj
Joints:
- added joint airskin_10_joint: type fixed, parent onrobot_rg6_base_link, child airskin_10, origin xyz=0.025 0 0.1 rpy=0 1.57 0
- added joint finger_joint: type revolute, parent onrobot_rg6_base_link, child left_outer_knuckle, origin xyz=0 -0.024112 0.136813 rpy=0 0 0, axis -1 0 0, limit lower=-0.628319 upper=0.628319 effort=1000 velocity=2.0
- added joint gripper_joint: type fixed, parent onrobot_rg6_base_link, child gripper_link, origin xyz=0. 0. 0.1667 rpy=0 0 1.57
- added joint jaws_joint: type prismatic, parent tool0, child jaws_link, origin xyz=0.0 0.0 0.0 rpy=0.0 0.0 0.0, axis 0.0 0.0 1.0, limit lower=0.0 upper=10.0 effort=1000.0 velocity=2.0
- added joint left_inner_finger_joint: type revolute, parent left_outer_knuckle, child left_inner_finger, origin xyz=0 -0.047334999999999995 0.064495 rpy=0 0 0, axis 1 0 0, limit lower=-0.872665 upper=0.872665 effort=1000 velocity=2.0, mimic joint=finger_joint multiplier=1 offset=0
- added joint left_inner_knuckle_joint: type revolute, parent onrobot_rg6_base_link, child left_inner_knuckle, origin xyz=0 -0.01272 0.159500 rpy=0 0 0.0, axis 1 0 0, limit lower=-0.628319 upper=0.628319 effort=1000 velocity=2.0, mimic joint=finger_joint multiplier=-1 offset=0
- added joint rg6_ur10_joint: type fixed, parent wrist_ft_sensor, child onrobot_rg6_base_link, origin xyz=0.0 0.0 0.0 rpy=0.0 1.57 0.0
- added joint right_inner_finger_joint: type revolute, parent right_outer_knuckle, child right_inner_finger, origin xyz=0 -0.047334999999999995 0.064495 rpy=0 0 0, axis 1 0 0, limit lower=-0.872665 upper=0.872665 effort=1000 velocity=2.0, mimic joint=finger_joint multiplier=1 offset=0
- added joint right_inner_knuckle_joint: type revolute, parent onrobot_rg6_base_link, child right_inner_knuckle, origin xyz=0 0.01272 0.159500 rpy=0 0 -3.141592653589793, axis 1 0 0, limit lower=-0.628319 upper=0.628319 effort=1000 velocity=2.0, mimic joint=finger_joint multiplier=-1 offset=0
- added joint right_outer_knuckle_joint: type revolute, parent onrobot_rg6_base_link, child right_outer_knuckle, origin xyz=0 0.024112 0.136813 rpy=0 0 3.141592653589793, axis 1 0 0, limit lower=-0.628319 upper=0.628319 effort=1000 velocity=2.0, mimic joint=finger_joint multiplier=-1 offset=0

File: src/ur10e_simulator/bullet_ros_ur/urdf/ur10e.urdf (robot description, URDF)
Before this commit: robot ur10e_robot, 37 links, 36 joints
Links:
- removed link airskin_10
- removed link backwall
- removed link ceiling
- removed link gripper_link
- removed link jaws_link
- removed link left_inner_finger
- removed link left_inner_knuckle
- removed link left_outer_knuckle
- removed link onrobot_rg6_base_link
- removed link right_inner_finger
- removed link right_inner_knuckle
- removed link right_outer_knuckle
Joints:
- removed joint airskin_10_joint
- removed joint backwall_joint
- removed joint ceiling_joint
- removed joint finger_joint
- removed joint gripper_joint
- removed joint jaws_joint
- removed joint left_inner_finger_joint
- removed joint left_inner_knuckle_joint
- removed joint rg6_ur10_joint
- removed joint right_inner_finger_joint
- removed joint right_inner_knuckle_joint
- removed joint right_outer_knuckle_joint
