Commit message: Fixed softhand visuals in ROS mode

File: src/ur10e_simulator/bullet_ros_ur/urdf/ur10e_softhand.urdf (robot description, URDF)
Before this commit: robot ur10e_robot, 63 links, 62 joints
Joints:
- joint qbhand_index_distal_joint: mimic joint=qbhand_synergy_joint multiplier=0.785 -> (none)
- joint qbhand_index_distal_virtual_joint: mimic joint=qbhand_index_distal_joint multiplier=1.0 -> (none)
- joint qbhand_index_knuckle_joint: mimic joint=qbhand_synergy_joint multiplier=-0.2 -> (none)
- joint qbhand_index_middle_joint: mimic joint=qbhand_synergy_joint multiplier=0.785 -> (none)
- joint qbhand_index_middle_virtual_joint: mimic joint=qbhand_index_middle_joint multiplier=1.0 -> (none)
- joint qbhand_index_proximal_joint: mimic joint=qbhand_synergy_joint multiplier=0.785 -> (none)
- joint qbhand_index_proximal_virtual_joint: mimic joint=qbhand_index_proximal_joint multiplier=1.0 -> (none)
- joint qbhand_little_distal_joint: mimic joint=qbhand_synergy_joint multiplier=0.785 -> (none)
- joint qbhand_little_distal_virtual_joint: mimic joint=qbhand_little_distal_joint multiplier=1.0 -> (none)
- joint qbhand_little_knuckle_joint: mimic joint=qbhand_synergy_joint multiplier=0.4 -> (none)
- joint qbhand_little_middle_joint: mimic joint=qbhand_synergy_joint multiplier=0.785 -> (none)
- joint qbhand_little_middle_virtual_joint: mimic joint=qbhand_little_middle_joint multiplier=1.0 -> (none)
- joint qbhand_little_proximal_joint: mimic joint=qbhand_synergy_joint multiplier=0.785 -> (none)
- joint qbhand_little_proximal_virtual_joint: mimic joint=qbhand_little_proximal_joint multiplier=1.0 -> (none)
- joint qbhand_middle_distal_joint: mimic joint=qbhand_synergy_joint multiplier=0.785 -> (none)
- joint qbhand_middle_distal_virtual_joint: mimic joint=qbhand_middle_distal_joint multiplier=1.0 -> (none)
- joint qbhand_middle_knuckle_joint: mimic joint=qbhand_synergy_joint multiplier=0.0 -> (none)
- joint qbhand_middle_middle_joint: mimic joint=qbhand_synergy_joint multiplier=0.785 -> (none)
- joint qbhand_middle_middle_virtual_joint: mimic joint=qbhand_middle_middle_joint multiplier=1.0 -> (none)
- joint qbhand_middle_proximal_joint: mimic joint=qbhand_synergy_joint multiplier=0.785 -> (none)
- joint qbhand_middle_proximal_virtual_joint: mimic joint=qbhand_middle_proximal_joint multiplier=1.0 -> (none)
- joint qbhand_ring_distal_joint: mimic joint=qbhand_synergy_joint multiplier=0.785 -> (none)
- joint qbhand_ring_distal_virtual_joint: mimic joint=qbhand_ring_distal_joint multiplier=1.0 -> (none)
- joint qbhand_ring_knuckle_joint: mimic joint=qbhand_synergy_joint multiplier=0.2 -> (none)
- joint qbhand_ring_middle_joint: mimic joint=qbhand_synergy_joint multiplier=0.785 -> (none)
- joint qbhand_ring_middle_virtual_joint: mimic joint=qbhand_ring_middle_joint multiplier=1.0 -> (none)
- joint qbhand_ring_proximal_joint: mimic joint=qbhand_synergy_joint multiplier=0.785 -> (none)
- joint qbhand_ring_proximal_virtual_joint: mimic joint=qbhand_ring_proximal_joint multiplier=1.0 -> (none)
- joint qbhand_thumb_distal_joint: mimic joint=qbhand_synergy_joint multiplier=0.785 -> (none)
- joint qbhand_thumb_distal_virtual_joint: mimic joint=qbhand_thumb_distal_joint multiplier=1.0 -> (none)
- joint qbhand_thumb_knuckle_joint: mimic joint=qbhand_synergy_joint multiplier=2.542 -> (none)
- joint qbhand_thumb_proximal_joint: mimic joint=qbhand_synergy_joint multiplier=0.785 -> (none)
- joint qbhand_thumb_proximal_virtual_joint: mimic joint=qbhand_thumb_proximal_joint multiplier=1.0 -> (none)
